File: schematics/uart_data_logger.kicad_sch (KiCad schematic)
At the start: 10 parts, among them J1 Micro_SD_Card, SW1 Start/Stop, U1 CH32V003F4P6

Commit message: updated schematics/layout.
Parts:
- removed D1: STATUS, LED_THT:LED_D3.0mm, symbol Device:LED
- removed J1: Micro_SD_Card, Connector_Card:microSD_HC_Hirose_DM3D-SF, symbol Connector:Micro_SD_Card
- removed SW1: Start/Stop, Button_Switch_THT:SW_PUSH_6mm_H4.3mm, symbol Switch:SW_Push
- added C5: 10uF, Capacitor_SMD:C_1206_3216Metric_Pad1.33x1.80mm_HandSolder, symbol Device:C_Small
- added J1: Micro_SD_Card, Connector_Card:microSD_HC_Hirose_DM3AT-SF-PEJM5, symbol Connector:Micro_SD_Card_Det_Hirose_DM3AT
- added J2: Conn_01x03, swk:1x03_THT_P2.54mm, symbol Connector_Generic:Conn_01x03
- added J3, J4: Conn_01x02, swk:1x02_THT_P2.54mm, symbol Connector_Generic:Conn_01x02
- added SW2: SW_Push_LED, swk:SW_Push_LED_AK104238, symbol swk:SW_Push_LED_AK104238
- added U3: AZ1117CH-3.3TRG1, Package_TO_SOT_SMD:SOT-223-3_TabPin2, symbol Regulator_Linear:AZ1117-3.3
- C1: value 220uf -> 100uF; footprint Capacitor_THT:CP_Radial_D7.5mm_P2.50mm -> Capacitor_SMD:C_1206_3216Metric_Pad1.33x1.80mm_HandSolder
- C2, C4: footprint Capacitor_THT:C_Disc_D4.3mm_W1.9mm_P5.00mm -> Capacitor_SMD:C_1206_3216Metric_Pad1.33x1.80mm_HandSolder
- C3: footprint Capacitor_THT:CP_Radial_D5.0mm_P2.00mm -> Capacitor_SMD:C_1206_3216Metric_Pad1.33x1.80mm_HandSolder
- R1, R2: footprint Resistor_THT:R_Axial_DIN0207_L6.3mm_D2.5mm_P7.62mm_Horizontal -> Resistor_SMD:R_1206_3216Metric_Pad1.30x1.75mm_HandSolder
- U1: footprint Package_SO:SOP-20_7.5x12.8mm_P1.27mm -> swk:TSSOP20
Connections:
- net +3.3V: now also J1.4 (VDD), J2.3 (Pin_3), U3.2 (VO)
- net COMM_Rx: now also J3.2 (Pin_2)
- net CS: now also J1.2 (DAT3/CD)
- net GND: now also C5.1, J1.6 (VSS), J2.2 (Pin_2), J3.1 (Pin_1), J4.1 (Pin_1), SW2.2, SW2.L2, U3.1 (GND)
- net MISO: now also J1.7 (DAT0)
- net MOSI: now also J1.3 (CMD)
- net PRG_SWIO: now also J4.2 (Pin_2)
- net SCK: now also J1.5 (CLK)
- net at U1.13 (PC3): now also SW2.1
- net at R2.1: now also SW2.L1
- new net: C5.2, J2.1 (Pin_1), U3.3 (VI)
